File: HW3/circuit_diagram.sch (EAGLE design)
At the start: 0 parts

Commit message: First elements and connections
Parts:
- added C1, C2, C3: (no value), resistor:C-US025-024X044
- added C4, C5: (no value), resistor:CPOL-USCT3216
- added LED1, LED2: (no value), led:LED3MM
- added R1, R2, R3, R4: (no value), resistor:R-US_0207/10
Connections:
- new net +3V3: C2.1, C3.1, C4.+, LED1.A, R2.1, R3.1
- new net GND: C1.2, C2.2, C4.-, C5.-, R1.2, R4.1
- new net N$1: LED1.C, R1.1
- new net N$2: LED2.C, R4.2
- new net N$3: R2.2
